Commit message: feat: enable odometry transformation and update launch configurations for multi-robot support

File: clearpath_ws/src/clearpath_common/clearpath_platform_description/urdf/generic/gazebo.urdf.xacro (robot description, xacro)
@@ -8,6 +8,6 @@
           <remapping>~/odom:=platform/odom</remapping>
           <remapping>~/cmd_vel_unstamped:=platform/cmd_vel_unstamped</remapping>
-          <remapping>/tf:=tf</remapping>
-          <remapping>/tf_static:=tf_static</remapping>
+          <remapping>/tf:=/tf</remapping>
+          <remapping>/tf_static:=/tf_static</remapping>
           <remapping>/diagnostics:=diagnostics</remapping>
           <remapping>/dynamic_joint_states:=platform/dynamic_joint_states</remapping>

File: clearpath_ws/src/clearpath_common/clearpath_sensors_description/urdf/velodyne_lidar.urdf.xacro (robot description, xacro)
@@ -6,4 +6,6 @@
                                              ang_res_v:=2.0 min_ang_v:=-0.261799 max_ang_v:=0.261799
                                              update_rate:=20 min_range:=0.9 max_range:=130.0">
+    <xacro:property name="robot_ns" value="$(arg namespace)"/>
+    <xacro:property name="frame_prefix" value="${robot_ns + '/' if robot_ns != '' else ''}"/>
     <link name="${name}_link">
       <inertial>
@@ -64,5 +66,5 @@
         <visualize>true</visualize>
         <always_on>true</always_on>
-        <ignition_frame_id>${name}_laser</ignition_frame_id>
+        <ignition_frame_id>${frame_prefix}${name}_laser</ignition_frame_id>
         <topic>$(arg namespace)/sensors/${name}/scan</topic>
         <lidar>
