Commit message: feat: add support for W200 body color configuration and update related robot YAML files

File: clearpath_ws/src/clearpath_common/clearpath_platform_description/urdf/w200/w200.urdf.xacro (robot description, xacro)
@@ -17,4 +17,5 @@
     <material name="warthog_olive"><color rgba="0.333 0.419 0.184 1.0"/></material>
     <material name="warthog_sand"><color rgba="0.86 0.75 0.54 1.0"/></material>
+    <material name="warthog_dark_olive"><color rgba="0.42 0.46 0.35 1.0"/></material>
     <!-- Variables -->
     <xacro:property name="wheel_radius" value="0.3" />

Commit message: feat: add namespace support for robot and frame prefix in URDF

File: clearpath_ws/src/clearpath_common/clearpath_platform_description/urdf/w200/w200.urdf.xacro (robot description, xacro)
@@ -135,4 +135,6 @@
       </xacro:w200_track>
     </xacro:if>
+    <xacro:property name="robot_ns" value="$(arg namespace)"/>
+    <xacro:property name="frame_prefix" value="${robot_ns + '/' if robot_ns != '' else ''}"/>
     <!-- Virtual Mounting Point -->
     <link name="default_mount"></link>
@@ -159,5 +161,5 @@
         <update_rate>50</update_rate>
         <visualize>true</visualize>
-        <ignition_frame_id>imu_0_link</ignition_frame_id>
+        <ignition_frame_id>${frame_prefix}imu_0_link</ignition_frame_id>
         <topic>$(arg namespace)/sensors/imu_0/data_raw</topic>
       </sensor>
