Commit message: feat: add inertial properties and collision geometries for canister links and base plate

File: robots/payloads/canisters.xacro (robot description, xacro)
@@ -23,4 +23,9 @@
   </material>
   <link name="base_plate">
+    <inertial>
+      <origin xyz="-0.006 0 0.0005" rpy="0 0 0"/>
+      <mass value="14.0"/>
+      <inertia ixx="0.430" ixy="0.0" ixz="0.0" iyy="0.760" iyz="0.0" izz="1.160"/>
+    </inertial>
     <visual>
       <origin xyz="0 0 0" rpy="0 0 0"/>
@@ -58,4 +63,28 @@
       <material name="mat_mid_detail"/>
     </visual>
+    <collision>
+      <origin xyz="0 0 0" rpy="0 0 0"/>
+      <geometry>
+        <box size="0.80 0.60 0.025"/>
+      </geometry>
+    </collision>
+    <collision>
+      <origin xyz="-0.02 0.24 -0.020" rpy="0 0 0"/>
+      <geometry>
+        <box size="0.70 0.05 0.030"/>
+      </geometry>
+    </collision>
+    <collision>
+      <origin xyz="-0.02 -0.24 -0.020" rpy="0 0 0"/>
+      <geometry>
+        <box size="0.70 0.05 0.030"/>
+      </geometry>
+    </collision>
+    <collision>
+      <origin xyz="0.24 0 0.0175" rpy="0 0 0"/>
+      <geometry>
+        <box size="0.14 0.50 0.006"/>
+      </geometry>
+    </collision>
   </link>
   <joint name="payload_mount_joint" type="fixed">
@@ -70,4 +99,9 @@
   </joint>
   <link name="lidar_tower">
+    <inertial>
+      <origin xyz="0 0 0.248" rpy="0 0 0"/>
+      <mass value="4.2"/>
+      <inertia ixx="0.089" ixy="0.0" ixz="0.0" iyy="0.089" iyz="0.0" izz="0.0048"/>
+    </inertial>
     <visual>
       <origin xyz="0 0 0.015" rpy="0 0 0"/>
@@ -105,4 +139,34 @@
       <material name="mat_canister_cap"/>
     </visual>
+    <collision>
+      <origin xyz="0 0 0.015" rpy="0 0 0"/>
+      <geometry>
+        <cylinder length="0.03" radius="0.06"/>
+      </geometry>
+    </collision>
+    <collision>
+      <origin xyz="0 0 0.05" rpy="0 0 0"/>
+      <geometry>
+        <cylinder length="0.04" radius="0.035"/>
+      </geometry>
+    </collision>
+    <collision>
+      <origin xyz="0 0 0.31" rpy="0 0 0"/>
+      <geometry>
+        <cylinder length="0.50" radius="0.022"/>
+      </geometry>
+    </collision>
+    <collision>
+      <origin xyz="0 0 0.45" rpy="0 0 0"/>
+      <geometry>
+        <cylinder length="0.03" radius="0.035"/>
+      </geometry>
+    </collision>
+    <collision>
+      <origin xyz="0 0 0.56" rpy="0 0 0"/>
+      <geometry>
+        <cylinder length="0.01" radius="0.060"/>
+      </geometry>
+    </collision>
   </link>
   <joint name="lidar_tower_joint" type="fixed">
@@ -111,5 +175,11 @@
     <origin xyz="0 0 0.0125" rpy="0 0 0"/>
   </joint>
-  <link name="turret_lidar_mount"/>
+  <link name="turret_lidar_mount">
+    <inertial>
+      <origin xyz="0 0 0" rpy="0 0 0"/>
+      <mass value="0.05"/>
+      <inertia ixx="0.00001" ixy="0.0" ixz="0.0" iyy="0.00001" iyz="0.0" izz="0.00001"/>
+    </inertial>
+  </link>
   <joint name="turret_lidar_mount_joint" type="fixed">
     <parent link="lidar_tower"/>
@@ -118,4 +188,9 @@
   </joint>
   <link name="payload_base_link">
+    <inertial>
+      <origin xyz="0.005 0 0.066" rpy="0 0 0"/>
+      <mass value="26.0"/>
+      <inertia ixx="0.640" ixy="0.0" ixz="0.0" iyy="0.150" iyz="0.0" izz="0.690"/>
+    </inertial>
     <visual>
       <origin xyz="0 0 0" rpy="0 0 0"/>
@@ -128,80 +203,151 @@
       <origin xyz="0 -0.19 0.07" rpy="1.5708 0 0"/>
       <geometry>
+        <cylinder length="0.19" radius="0.10"/>
+      </geometry>
+      <material name="mat_soft_panel"/>
+    </visual>
+    <visual>
+      <origin xyz="0 0.19 0.07" rpy="1.5708 0 0"/>
+      <geometry>
+        <cylinder length="0.19" radius="0.10"/>
+      </geometry>
+      <material name="mat_soft_panel"/>
+    </visual>
+    <visual>
+      <origin xyz="0 0 0.085" rpy="0 0 0"/>
+      <geometry>
+        <box size="0.16 0.44 0.05"/>
+      </geometry>
+      <material name="mat_soft_panel"/>
+    </visual>
+    <visual>
+      <origin xyz="0.055 0 0.040" rpy="0 0 0"/>
+      <geometry>
+        <box size="0.03 0.52 0.06"/>
+      </geometry>
+      <material name="mat_mid_detail"/>
+    </visual>
+    <visual>
+      <origin xyz="-0.055 0 0.040" rpy="0 0 0"/>
+      <geometry>
+        <box size="0.03 0.52 0.06"/>
+      </geometry>
+      <material name="mat_mid_detail"/>
+    </visual>
+    <visual>
+      <origin xyz="0.035 0.19 0.105" rpy="0 0.45 0"/>
+      <geometry>
+        <box size="0.10 0.06 0.05"/>
+      </geometry>
+      <material name="mat_dark_detail"/>
+    </visual>
+    <visual>
+      <origin xyz="0.035 -0.19 0.105" rpy="0 0.45 0"/>
+      <geometry>
+        <box size="0.10 0.06 0.05"/>
+      </geometry>
+      <material name="mat_dark_detail"/>
+    </visual>
+    <visual>
+      <origin xyz="-0.045 0.19 0.102" rpy="0 -0.35 0"/>
+      <geometry>
+        <box size="0.09 0.06 0.045"/>
+      </geometry>
+      <material name="mat_mid_detail"/>
+    </visual>
+    <visual>
+      <origin xyz="-0.045 -0.19 0.102" rpy="0 -0.35 0"/>
+      <geometry>
+        <box size="0.09 0.06 0.045"/>
+      </geometry>
+      <material name="mat_mid_detail"/>
+    </visual>
+    <visual>
+      <origin xyz="0.07 0 0.095" rpy="0 0 0"/>
+      <geometry>
+        <box size="0.03 0.40 0.02"/>
+      </geometry>
+      <material name="mat_canister_cap"/>
+    </visual>
+    <visual>
+      <origin xyz="-0.085 0 0.070" rpy="0 0 0"/>
+      <geometry>
+        <box size="0.02 0.36 0.05"/>
+      </geometry>
+      <material name="mat_dark_detail"/>
+    </visual>
+    <collision>
+      <origin xyz="0 0 0" rpy="0 0 0"/>
+      <geometry>
+        <box size="0.20 0.58 0.10"/>
+      </geometry>
+    </collision>
+    <collision>
+      <origin xyz="0 -0.19 0.07" rpy="1.5708 0 0"/>
+      <geometry>
         <cylinder length="0.20" radius="0.10"/>
       </geometry>
-      <material name="mat_base"/>
-    </visual>
-    <visual>
+    </collision>
+    <collision>
       <origin xyz="0 0.19 0.07" rpy="1.5708 0 0"/>
       <geometry>
         <cylinder length="0.20" radius="0.10"/>
       </geometry>
-      <material name="mat_base"/>
-    </visual>
-    <visual>
-      <origin xyz="0 0 0.085" rpy="0 0 0"/>
-      <geometry>
-        <box size="0.16 0.44 0.05"/>
-      </geometry>
-      <material name="mat_soft_panel"/>
-    </visual>
-    <visual>
+    </collision>
+    <collision>
       <origin xyz="0.055 0 0.040" rpy="0 0 0"/>
       <geometry>
         <box size="0.03 0.52 0.06"/>
       </geometry>
-      <material name="mat_mid_detail"/>
-    </visual>
-    <visual>
+    </collision>
+    <collision>
       <origin xyz="-0.055 0 0.040" rpy="0 0 0"/>
       <geometry>
         <box size="0.03 0.52 0.06"/>
       </geometry>
-      <material name="mat_mid_detail"/>
-    </visual>
-    <visual>
+    </collision>
+    <collision>
       <origin xyz="0.035 0.19 0.105" rpy="0 0.45 0"/>
       <geometry>
         <box size="0.10 0.06 0.05"/>
       </geometry>
-      <material name="mat_dark_detail"/>
-    </visual>
-    <visual>
+    </collision>
+    <collision>
       <origin xyz="0.035 -0.19 0.105" rpy="0 0.45 0"/>
       <geometry>
         <box size="0.10 0.06 0.05"/>
       </geometry>
-      <material name="mat_dark_detail"/>
-    </visual>
-    <visual>
+    </collision>
+    <collision>
       <origin xyz="-0.045 0.19 0.102" rpy="0 -0.35 0"/>
       <geometry>
         <box size="0.09 0.06 0.045"/>
       </geometry>
-      <material name="mat_mid_detail"/>
-    </visual>
-    <visual>
+    </collision>
+    <collision>
       <origin xyz="-0.045 -0.19 0.102" rpy="0 -0.35 0"/>
       <geometry>
         <box size="0.09 0.06 0.045"/>
       </geometry>
-      <material name="mat_mid_detail"/>
-    </visual>
-    <visual>
+    </collision>
+    <collision>
       <origin xyz="0.07 0 0.095" rpy="0 0 0"/>
       <geometry>
         <box size="0.03 0.40 0.02"/>
       </geometry>
-      <material name="mat_canister_cap"/>
-    </visual>
-    <visual>
+    </collision>
+    <collision>
       <origin xyz="-0.085 0 0.070" rpy="0 0 0"/>
       <geometry>
         <box size="0.02 0.36 0.05"/>
       </geometry>
-      <material name="mat_dark_detail"/>
-    </visual>
+    </collision>
   </link>
   <link name="left_canister_link">
+    <inertial>
+      <origin xyz="0.325 0 0.10" rpy="0 0 0"/>
+      <mass value="21.0"/>
+      <inertia ixx="0.067" ixy="0.0" ixz="0.0" iyy="1.90" iyz="0.0" izz="1.90"/>
+    </inertial>
     <visual>
       <origin xyz="0.30 0 0.10" rpy="0 1.57079632679 0"/>
@@ -209,5 +355,5 @@
         <cylinder length="1.00" radius="0.09"/>
       </geometry>
-      <material name="mat_canister_body"/>
+      <material name="mat_canister_cap"/>
     </visual>
     <visual>
@@ -218,6 +364,23 @@
       <material name="mat_canister_cap"/>
     </visual>
+    <collision>
+      <origin xyz="0.30 0 0.10" rpy="0 1.57079632679 0"/>
+      <geometry>
+        <cylinder length="1.00" radius="0.09"/>
+      </geometry>
+    </collision>
+    <collision>
+      <origin xyz="0.77 0 0.10" rpy="0 1.57079632679 0"/>
+      <geometry>
+        <cylinder length="0.10" radius="0.10"/>
+      </geometry>
+    </collision>
   </link>
   <link name="right_canister_link">
+    <inertial>
+      <origin xyz="0.325 0 0.10" rpy="0 0 0"/>
+      <mass value="21.0"/>
+      <inertia ixx="0.067" ixy="0.0" ixz="0.0" iyy="1.90" iyz="0.0" izz="1.90"/>
+    </inertial>
     <visual>
       <origin xyz="0.30 0 0.10" rpy="0 1.57079632679 0"/>
@@ -225,5 +388,5 @@
         <cylinder length="1.00" radius="0.09"/>
       </geometry>
-      <material name="mat_canister_body"/>
+      <material name="mat_canister_cap"/>
     </visual>
     <visual>
@@ -234,4 +397,16 @@
       <material name="mat_canister_cap"/>
     </visual>
+    <collision>
+      <origin xyz="0.30 0 0.10" rpy="0 1.57079632679 0"/>
+      <geometry>
+        <cylinder length="1.00" radius="0.09"/>
+      </geometry>
+    </collision>
+    <collision>
+      <origin xyz="0.77 0 0.10" rpy="0 1.57079632679 0"/>
+      <geometry>
+        <cylinder length="0.10" radius="0.10"/>
+      </geometry>
+    </collision>
   </link>
   <joint name="left_canister_joint" type="revolute">

Commit message: feat: add dynamics properties to canister joints and Gazebo plugins for position control

File: robots/payloads/canisters.xacro (robot description, xacro)
@@ -416,4 +416,5 @@
     <axis xyz="0 1 0"/>
     <limit lower="-0.87" upper="0" effort="10" velocity="1.0"/>
+    <dynamics damping="1.0" friction="0.1"/>
   </joint>
   <joint name="right_canister_joint" type="revolute">
@@ -423,4 +424,33 @@
     <axis xyz="0 1 0"/>
     <limit lower="-0.87" upper="0" effort="10" velocity="1.0"/>
-  </joint>
+    <dynamics damping="1.0" friction="0.1"/>
+  </joint>
+  <gazebo>
+    <plugin filename="gz-sim-joint-position-controller-system"
+            name="gz::sim::systems::JointPositionController">
+      <joint_name>left_canister_joint</joint_name>
+      <joint_index>0</joint_index>
+      <p_gain>80.0</p_gain>
+      <i_gain>0.0</i_gain>
+      <d_gain>8.0</d_gain>
+      <i_max>0.0</i_max>
+      <i_min>0.0</i_min>
+      <cmd_max>10.0</cmd_max>
+      <cmd_min>-10.0</cmd_min>
+      <topic>/left_canister/cmd_pos</topic>
+    </plugin>
+    <plugin filename="gz-sim-joint-position-controller-system"
+            name="gz::sim::systems::JointPositionController">
+      <joint_name>right_canister_joint</joint_name>
+      <joint_index>0</joint_index>
+      <p_gain>80.0</p_gain>
+      <i_gain>0.0</i_gain>
+      <d_gain>8.0</d_gain>
+      <i_max>0.0</i_max>
+      <i_min>0.0</i_min>
+      <cmd_max>10.0</cmd_max>
+      <cmd_min>-10.0</cmd_min>
+      <topic>/right_canister/cmd_pos</topic>
+    </plugin>
+  </gazebo>
 </robot>

Commit message: feat: add ripgrep installation to AMD64 and ARM64 Dockerfiles; update canister collision geometries and joint configurations

File: robots/payloads/canisters.xacro (robot description, xacro)
@@ -69,22 +69,4 @@
       </geometry>
     </collision>
-    <collision>
-      <origin xyz="-0.02 0.24 -0.020" rpy="0 0 0"/>
-      <geometry>
-        <box size="0.70 0.05 0.030"/>
-      </geometry>
-    </collision>
-    <collision>
-      <origin xyz="-0.02 -0.24 -0.020" rpy="0 0 0"/>
-      <geometry>
-        <box size="0.70 0.05 0.030"/>
-      </geometry>
-    </collision>
-    <collision>
-      <origin xyz="0.24 0 0.0175" rpy="0 0 0"/>
-      <geometry>
-        <box size="0.14 0.50 0.006"/>
-      </geometry>
-    </collision>
   </link>
   <joint name="payload_mount_joint" type="fixed">
@@ -140,31 +122,7 @@
     </visual>
     <collision>
-      <origin xyz="0 0 0.015" rpy="0 0 0"/>
-      <geometry>
-        <cylinder length="0.03" radius="0.06"/>
-      </geometry>
-    </collision>
-    <collision>
-      <origin xyz="0 0 0.05" rpy="0 0 0"/>
-      <geometry>
-        <cylinder length="0.04" radius="0.035"/>
-      </geometry>
-    </collision>
-    <collision>
-      <origin xyz="0 0 0.31" rpy="0 0 0"/>
-      <geometry>
-        <cylinder length="0.50" radius="0.022"/>
-      </geometry>
-    </collision>
-    <collision>
-      <origin xyz="0 0 0.45" rpy="0 0 0"/>
-      <geometry>
-        <cylinder length="0.03" radius="0.035"/>
-      </geometry>
-    </collision>
-    <collision>
-      <origin xyz="0 0 0.56" rpy="0 0 0"/>
-      <geometry>
-        <cylinder length="0.01" radius="0.060"/>
+      <origin xyz="0 0 0.28" rpy="0 0 0"/>
+      <geometry>
+        <cylinder length="0.58" radius="0.06"/>
       </geometry>
     </collision>
@@ -278,67 +236,7 @@
     </visual>
     <collision>
-      <origin xyz="0 0 0" rpy="0 0 0"/>
-      <geometry>
-        <box size="0.20 0.58 0.10"/>
-      </geometry>
-    </collision>
-    <collision>
-      <origin xyz="0 -0.19 0.07" rpy="1.5708 0 0"/>
-      <geometry>
-        <cylinder length="0.20" radius="0.10"/>
-      </geometry>
-    </collision>
-    <collision>
-      <origin xyz="0 0.19 0.07" rpy="1.5708 0 0"/>
-      <geometry>
-        <cylinder length="0.20" radius="0.10"/>
-      </geometry>
-    </collision>
-    <collision>
-      <origin xyz="0.055 0 0.040" rpy="0 0 0"/>
-      <geometry>
-        <box size="0.03 0.52 0.06"/>
-      </geometry>
-    </collision>
-    <collision>
-      <origin xyz="-0.055 0 0.040" rpy="0 0 0"/>
-      <geometry>
-        <box size="0.03 0.52 0.06"/>
-      </geometry>
-    </collision>
-    <collision>
-      <origin xyz="0.035 0.19 0.105" rpy="0 0.45 0"/>
-      <geometry>
-        <box size="0.10 0.06 0.05"/>
-      </geometry>
-    </collision>
-    <collision>
-      <origin xyz="0.035 -0.19 0.105" rpy="0 0.45 0"/>
-      <geometry>
-        <box size="0.10 0.06 0.05"/>
-      </geometry>
-    </collision>
-    <collision>
-      <origin xyz="-0.045 0.19 0.102" rpy="0 -0.35 0"/>
-      <geometry>
-        <box size="0.09 0.06 0.045"/>
-      </geometry>
-    </collision>
-    <collision>
-      <origin xyz="-0.045 -0.19 0.102" rpy="0 -0.35 0"/>
-      <geometry>
-        <box size="0.09 0.06 0.045"/>
-      </geometry>
-    </collision>
-    <collision>
-      <origin xyz="0.07 0 0.095" rpy="0 0 0"/>
-      <geometry>
-        <box size="0.03 0.40 0.02"/>
-      </geometry>
-    </collision>
-    <collision>
-      <origin xyz="-0.085 0 0.070" rpy="0 0 0"/>
-      <geometry>
-        <box size="0.02 0.36 0.05"/>
+      <origin xyz="0 0 0.06" rpy="0 0 0"/>
+      <geometry>
+        <box size="0.20 0.58 0.18"/>
       </geometry>
     </collision>
@@ -346,7 +244,7 @@
   <link name="left_canister_link">
     <inertial>
-      <origin xyz="0.325 0 0.10" rpy="0 0 0"/>
-      <mass value="21.0"/>
-      <inertia ixx="0.067" ixy="0.0" ixz="0.0" iyy="1.90" iyz="0.0" izz="1.90"/>
+      <origin xyz="0.35 0 0.10" rpy="0 0 0"/>
+      <mass value="5.0"/>
+      <inertia ixx="0.015" ixy="0.0" ixz="0.0" iyy="0.60" iyz="0.0" izz="0.60"/>
     </inertial>
     <visual>
@@ -355,5 +253,5 @@
         <cylinder length="1.00" radius="0.09"/>
       </geometry>
-      <material name="mat_canister_cap"/>
+      <material name="mat_canister_body"/>
     </visual>
     <visual>
@@ -365,46 +263,34 @@
     </visual>
     <collision>
+      <origin xyz="0.35 0 0.10" rpy="0 1.57079632679 0"/>
+      <geometry>
+        <cylinder length="1.10" radius="0.10"/>
+      </geometry>
+    </collision>
+  </link>
+  <link name="right_canister_link">
+    <inertial>
+      <origin xyz="0.35 0 0.10" rpy="0 0 0"/>
+      <mass value="5.0"/>
+      <inertia ixx="0.015" ixy="0.0" ixz="0.0" iyy="0.60" iyz="0.0" izz="0.60"/>
+    </inertial>
+    <visual>
       <origin xyz="0.30 0 0.10" rpy="0 1.57079632679 0"/>
       <geometry>
         <cylinder length="1.00" radius="0.09"/>
       </geometry>
-    </collision>
-    <collision>
+      <material name="mat_canister_body"/>
+    </visual>
+    <visual>
       <origin xyz="0.77 0 0.10" rpy="0 1.57079632679 0"/>
       <geometry>
         <cylinder length="0.10" radius="0.10"/>
       </geometry>
-    </collision>
-  </link>
-  <link name="right_canister_link">
-    <inertial>
-      <origin xyz="0.325 0 0.10" rpy="0 0 0"/>
-      <mass value="21.0"/>
-      <inertia ixx="0.067" ixy="0.0" ixz="0.0" iyy="1.90" iyz="0.0" izz="1.90"/>
-    </inertial>
-    <visual>
-      <origin xyz="0.30 0 0.10" rpy="0 1.57079632679 0"/>
-      <geometry>
-        <cylinder length="1.00" radius="0.09"/>
-      </geometry>
-      <material name="mat_canister_cap"/>
-    </visual>
-    <visual>
-      <origin xyz="0.77 0 0.10" rpy="0 1.57079632679 0"/>
-      <geometry>
-        <cylinder length="0.10" radius="0.10"/>
-      </geometry>
-      <material name="mat_canister_cap"/>
-    </visual>
-    <collision>
-      <origin xyz="0.30 0 0.10" rpy="0 1.57079632679 0"/>
-      <geometry>
-        <cylinder length="1.00" radius="0.09"/>
-      </geometry>
-    </collision>
-    <collision>
-      <origin xyz="0.77 0 0.10" rpy="0 1.57079632679 0"/>
-      <geometry>
-        <cylinder length="0.10" radius="0.10"/>
+      <material name="mat_canister_cap"/>
+    </visual>
+    <collision>
+      <origin xyz="0.35 0 0.10" rpy="0 1.57079632679 0"/>
+      <geometry>
+        <cylinder length="1.10" radius="0.10"/>
       </geometry>
     </collision>
@@ -414,7 +300,7 @@
     <child link="left_canister_link"/>
     <origin xyz="0 0.19 0.05" rpy="0 0 0"/>
-    <axis xyz="0 1 0"/>
-    <limit lower="-0.87" upper="0" effort="10" velocity="1.0"/>
-    <dynamics damping="1.0" friction="0.1"/>
+    <axis xyz="0 -1 0"/>
+    <limit lower="0" upper="0.87" effort="20" velocity="1.2"/>
+    <dynamics damping="1.5" friction="0.1"/>
   </joint>
   <joint name="right_canister_joint" type="revolute">
@@ -422,35 +308,50 @@
     <child link="right_canister_link"/>
     <origin xyz="0 -0.19 0.05" rpy="0 0 0"/>
-    <axis xyz="0 1 0"/>
-    <limit lower="-0.87" upper="0" effort="10" velocity="1.0"/>
-    <dynamics damping="1.0" friction="0.1"/>
-  </joint>
-  <gazebo>
-    <plugin filename="gz-sim-joint-position-controller-system"
-            name="gz::sim::systems::JointPositionController">
-      <joint_name>left_canister_joint</joint_name>
-      <joint_index>0</joint_index>
-      <p_gain>80.0</p_gain>
-      <i_gain>0.0</i_gain>
-      <d_gain>8.0</d_gain>
-      <i_max>0.0</i_max>
-      <i_min>0.0</i_min>
-      <cmd_max>10.0</cmd_max>
-      <cmd_min>-10.0</cmd_min>
-      <topic>/left_canister/cmd_pos</topic>
-    </plugin>
-    <plugin filename="gz-sim-joint-position-controller-system"
-            name="gz::sim::systems::JointPositionController">
-      <joint_name>right_canister_joint</joint_name>
-      <joint_index>0</joint_index>
-      <p_gain>80.0</p_gain>
-      <i_gain>0.0</i_gain>
-      <d_gain>8.0</d_gain>
-      <i_max>0.0</i_max>
-      <i_min>0.0</i_min>
-      <cmd_max>10.0</cmd_max>
-      <cmd_min>-10.0</cmd_min>
-      <topic>/right_canister/cmd_pos</topic>
-    </plugin>
-  </gazebo>
+    <axis xyz="0 -1 0"/>
+    <limit lower="0" upper="0.87" effort="20" velocity="1.2"/>
+    <dynamics damping="1.5" friction="0.1"/>
+  </joint>
+  <xacro:if value="$(arg is_sim)">
+    <ros2_control name="canister_state_hardware" type="system">
+      <hardware>
+        <plugin>ign_ros2_control/IgnitionSystem</plugin>
+      </hardware>
+      <joint name="left_canister_joint">
+        <state_interface name="position"/>
+        <state_interface name="velocity"/>
+      </joint>
+      <joint name="right_canister_joint">
+        <state_interface name="position"/>
+        <state_interface name="velocity"/>
+      </joint>
+    </ros2_control>
+  </xacro:if>
+<gazebo>
+  <plugin filename="gz-sim-joint-position-controller-system"
+          name="ignition::gazebo::systems::JointPositionController">
+    <joint_name>left_canister_joint</joint_name>
+    <joint_index>0</joint_index>
+    <p_gain>60.0</p_gain>
+    <i_gain>0.0</i_gain>
+    <d_gain>6.0</d_gain>
+    <i_max>0.0</i_max>
+    <i_min>0.0</i_min>
+    <cmd_max>20.0</cmd_max>
+    <cmd_min>-20.0</cmd_min>
+    <topic>/left_canister/cmd_pos</topic>
+  </plugin>
+  <plugin filename="gz-sim-joint-position-controller-system"
+          name="ignition::gazebo::systems::JointPositionController">
+    <joint_name>right_canister_joint</joint_name>
+    <joint_index>0</joint_index>
+    <p_gain>60.0</p_gain>
+    <i_gain>0.0</i_gain>
+    <d_gain>6.0</d_gain>
+    <i_max>0.0</i_max>
+    <i_min>0.0</i_min>
+    <cmd_max>20.0</cmd_max>
+    <cmd_min>-20.0</cmd_min>
+    <topic>/right_canister/cmd_pos</topic>
+  </plugin>
+</gazebo>
 </robot>
