Commit message: feat: add turret camera support with configuration for Intel RealSense

File: robots/payloads/canisters.xacro (robot description, xacro)
@@ -108,5 +108,5 @@
     </visual>
     <visual>
-      <origin xyz="0 0 0.45" rpy="0 0 0"/>
+      <origin xyz="0 0 0.5" rpy="0 0 0"/>
       <geometry>
         <cylinder length="0.03" radius="0.035"/>
@@ -144,4 +144,50 @@
     <child link="turret_lidar_mount"/>
     <origin xyz="0 0 0.565" rpy="0 0 0"/>
+  </joint>
+  <link name="turret_camera_support">
+    <inertial>
+      <origin xyz="0.060 0 0" rpy="0 0 0"/>
+      <mass value="0.10"/>
+      <inertia ixx="0.00010" ixy="0.0" ixz="0.0"
+              iyy="0.00020" iyz="0.0"
+              izz="0.00020"/>
+    </inertial>
+    <visual>
+      <origin xyz="0.055 0 0" rpy="0 0 0"/>
+      <geometry>
+        <box size="0.110 0.018 0.018"/>
+      </geometry>
+      <material name="mat_mid_detail"/>
+    </visual>
+    <visual>
+      <origin xyz="0.112 0 0" rpy="0 0 0"/>
+      <geometry>
+        <box size="0.004 0.050 0.034"/>
+      </geometry>
+      <material name="mat_dark_detail"/>
+    </visual>
+    <collision>
+      <origin xyz="0.058 0 0" rpy="0 0 0"/>
+      <geometry>
+        <box size="0.116 0.050 0.034"/>
+      </geometry>
+    </collision>
+  </link>
+  <joint name="turret_camera_support_joint" type="fixed">
+    <parent link="lidar_tower"/>
+    <child link="turret_camera_support"/>
+    <origin xyz="0.025 0 0.50" rpy="0 0 0"/>
+  </joint>
+  <link name="turret_camera_mount">
+    <inertial>
+      <origin xyz="0 0 0" rpy="0 0 0"/>
+      <mass value="0.05"/>
+      <inertia ixx="0.00001" ixy="0.0" ixz="0.0" iyy="0.00001" iyz="0.0" izz="0.00001"/>
+    </inertial>
+  </link>
+  <joint name="turret_camera_mount_joint" type="fixed">
+    <parent link="turret_camera_support"/>
+    <child link="turret_camera_mount"/>
+    <origin xyz="0.125 0 -0.01" rpy="0 0 0"/>
   </joint>
   <link name="payload_base_link">
