Commit message: feat: add robot_namespace parameter to Intel Realsense URDF and update optical frame ID reference

File: clearpath_ws/src/clearpath_common/clearpath_sensors_description/urdf/intel_realsense.urdf.xacro (robot description, xacro)
@@ -2,5 +2,6 @@
 <robot xmlns:xacro="http://ros.org/wiki/xacro">
   <xacro:macro name="intel_realsense" params="name parent_link *origin
-                                              update_rate:=30.0 image_height:=480 image_width:=640">
+                                              update_rate:=30.0 image_height:=480 image_width:=640 robot_namespace:=''">
+    <xacro:property name="color_optical_frame_id" value="${robot_namespace + '/' + name + '_color_optical_frame' if robot_namespace else name + '_color_optical_frame'}"/>
     <xacro:macro name="sensor_d435"
                  params="parent *origin name:=camera
@@ -149,5 +150,5 @@
           </clip>
           <ignition_frame_id>${name}_link</ignition_frame_id>
-          <optical_frame_id>${name}_color_optical_frame</optical_frame_id>
+          <optical_frame_id>${color_optical_frame_id}</optical_frame_id>
         </camera>
         <always_on>1</always_on>
